File: Kicad-RingPush/V1/RingPush-PMOD.sch (KiCad schematic (older format))
At the start: 37 parts, among them Q1 2N7002, Q2 2N7002, SW1 Rotary_Encoder_Switch, U1 74HC595

Commit message: Add libs
Parts:
- PMOD1: symbol PMOD:PMOD-Device-x2-Type-1A-GPIO -> RingPush-PMOD-rescue:PMOD-Device-x2-Type-1A-GPIO-PMOD
Changed lines of the file:
@@
 $EndComp
 $Comp
-L PMOD:PMOD-Device-x2-Type-1A-GPIO PMOD1
+L RingPush-PMOD-rescue:PMOD-Device-x2-Type-1A-GPIO-PMOD PMOD1
 U 1 1 607AB0A6
 P 3700 2850
